File: KiCAD/PUMA_PCB_REV1/_autosave-PUMA_PCB_REV1.kicad_pcb (KiCad board)
At the start: 4 copper layers, 141.7 x 141.5 mm, 49 parts, among them J1 SAMTEC-TMM-116-01-X-D-SM, U1 MICROFC-30035-SMT-TR1, U10 MICROFC-30035-SMT-TR1, U11 MICROFC-30035-SMT-TR1, U12 MICROFC-30035-SMT-TR1, U13 MICROFC-30035-SMT-TR1, U14 MICROFC-30035-SMT-TR1, U15 MICROFC-30035-SMT-TR1, U16 MICROFC-30035-SMT-TR1, U2 MICROFC-30035-SMT-TR1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

Commit message: added grounding zone first attempt
Parts:
- added H1: MountingHole, MountingHole:MountingHole_3.2mm_M3, F.Cu at (67.1, 169.9)
- added H2: MountingHole, MountingHole:MountingHole_3.2mm_M3, F.Cu at (58.4, 143.8)
- added H3: MountingHole, MountingHole:MountingHole_3.2mm_M3, F.Cu at (65.9, 118.8)
- added H4: MountingHole, MountingHole:MountingHole_3.2mm_M3, F.Cu at (78.4, 95.8)
- added H5: MountingHole, MountingHole:MountingHole_3.2mm_M3, F.Cu at (95.0, 75.7)
- added H6: MountingHole, MountingHole:MountingHole_3.2mm_M3, F.Cu at (115.2, 59.1)
- added H7: MountingHole, MountingHole:MountingHole_3.2mm_M3, F.Cu at (138.1, 46.8)
- added H8: MountingHole, MountingHole:MountingHole_3.2mm_M3, F.Cu at (163.2, 39.2)
- added H9: MountingHole, MountingHole:MountingHole_3.2mm_M3, F.Cu at (189.1, 36.6)
Connections:
- J1 pad 10: unconnected-(J1-Pad10) -> GND
- J1 pad 11: unconnected-(J1-Pad11) -> GND
- J1 pad 14: unconnected-(J1-Pad14) -> GND
- J1 pad 15: unconnected-(J1-Pad15) -> GND
- J1 pad 18: unconnected-(J1-Pad18) -> GND
- J1 pad 19: unconnected-(J1-Pad19) -> GND
- J1 pad 2: unconnected-(J1-Pad2) -> GND
- J1 pad 22: unconnected-(J1-Pad22) -> GND
- J1 pad 23: unconnected-(J1-Pad23) -> GND
- J1 pad 26: unconnected-(J1-Pad26) -> GND
- J1 pad 27: unconnected-(J1-Pad27) -> GND
- J1 pad 3: unconnected-(J1-Pad3) -> GND
- J1 pad 30: unconnected-(J1-Pad30) -> GND
- J1 pad 31: unconnected-(J1-Pad31) -> GND
- J1 pad 6: unconnected-(J1-Pad6) -> GND
- J1 pad 7: unconnected-(J1-Pad7) -> GND
- U1 pad 2: GND -> unconnected-(U1-Pad2)
- U10 pad 2: GND -> unconnected-(U10-Pad2)
- U11 pad 2: GND -> unconnected-(U11-Pad2)
- U12 pad 2: GND -> unconnected-(U12-Pad2)
- U13 pad 2: GND -> unconnected-(U13-Pad2)
- U14 pad 2: GND -> unconnected-(U14-Pad2)
- U15 pad 2: GND -> unconnected-(U15-Pad2)
- U16 pad 2: GND -> unconnected-(U16-Pad2)
- U2 pad 2: GND -> unconnected-(U2-Pad2)
- U3 pad 2: GND -> unconnected-(U3-Pad2)
- U4 pad 2: GND -> unconnected-(U4-Pad2)
- U5 pad 2: GND -> unconnected-(U5-Pad2)
- U6 pad 2: GND -> unconnected-(U6-Pad2)
- U7 pad 2: GND -> unconnected-(U7-Pad2)
- U8 pad 2: GND -> unconnected-(U8-Pad2)
- U9 pad 2: GND -> unconnected-(U9-Pad2)
Routing:
- net PW_3: track 60.4 -> 63.4 mm
- net PW_4: track 59.6 -> 61.5 mm
- net Net-(C15-Pad1): track 7.26 -> 7.87 mm, vias 1 -> 2
- net Net-(C9-Pad1): track 5.24 -> 5.80 mm
- net GND: track 0.82 -> 1.25 mm, vias 0 -> 40
- net (no net): vias 14 -> 0
- added copper zone on B.Cu, net GND
- added copper zone on F.Cu, net GND
- added copper zone on In1.Cu, net GND
- added copper zone on In2.Cu, net GND
