File: KiCAD/PUMA_PCB_REV1/_autosave-PUMA_PCB_REV1.kicad_pcb (KiCad board)
At the start: 4 copper layers, 141.7 x 141.5 mm, 59 parts, among them J1 SAMTEC-TMM-116-01-X-D-SM, J2 1778764, U1 MICROFC-30035-SMT-TR1, U10 MICROFC-30035-SMT-TR1, U11 MICROFC-30035-SMT-TR1, U12 MICROFC-30035-SMT-TR1, U13 MICROFC-30035-SMT-TR1, U14 MICROFC-30035-SMT-TR1, U15 MICROFC-30035-SMT-TR1, U16 MICROFC-30035-SMT-TR1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

Commit message: connect HV - problem in the center of board
Parts:
- moved R2 0.37 mm to (60.3, 151.6)
Connections:
- J2 pad 2: GND -> unconnected-(J2-Pad2)
Routing:
- net +HV: track 7.39 -> 0.00 mm
