File: KiCAD/PUMA_PCB_REV2/_autosave-PUMA_PCB_REV2.kicad_pcb (KiCad board)
At the start: 4 copper layers, 26.9 x 15.6 mm, 20 parts, among them J1 87832-0411, J2 CONMHF4-SMD-G-T, J3 CONMHF4-SMD-G-T, U1 MICROFC-30035-SMT-TR1, U2 MICROFC-30035-SMT-TR1

Commit message: changed holes
Parts:
- H2: footprint MountingHole:CastellatedHole -> MountingHole:MountingHole_2.5mm
- H3, H4: footprint MountingHole:Castelated_Hold_Right -> MountingHole:MountingHole_2.5mm
- moved H2 0.07 mm to (87.8, 95.5)
Connections:
- H1 pad : GND -> (no net)
